File: 3.3v_reg.sch (KiCad schematic (older format))
At the start: 5 parts, among them U4.1 LM5165Y

Commit message: updated PDU schematic with footprints
Parts:
- removed R4.1: 100k, symbol Device:R
- removed U4.1: LM5165Y, Package_SON:Texas_S-PVSON-N10_ThermalVias, symbol PowerDistributionUnit-rescue:LM5165Y-Regulator_Switching
- added R4.1: 1M, Resistor_SMD:R_01005_0402Metric, symbol PowerDistributionUnit-rescue:R-Device
- added U4.1: TPS62086, TPS62086LTR:TPS62086RLTR, symbol PDU_PROTOTYPE:TPS62086
- C4.1: value 13uF -> 10uF; footprint (none) -> Capacitor_SMD:C_0805_2012Metric; symbol Device:C -> PowerDistributionUnit-rescue:C-Device
- C4.2: footprint (none) -> Capacitor_SMD:C_0805_2012Metric; symbol Device:C -> PowerDistributionUnit-rescue:C-Device
- L4.1: value 373uH -> 0.47uH; symbol Device:L -> PowerDistributionUnit-rescue:L-Device
Connections:
- net labels added: GNDA
- wire segments 18 -> 29
