File: 5v_reg.sch (KiCad schematic (older format))
At the start: 11 parts, among them U3.1 LMR61428

Commit message: updated PDU schematic with footprints
Parts:
- removed C3.1: 22u, symbol Device:CP1
- removed C3.2: 39p, symbol Device:CP1
- removed C3.3: 1u, symbol Device:CP1
- removed C3.4: 68u, symbol Device:CP1
- removed D3.1: D_Zener, symbol Device:D_Zener
- removed L3.1: 6.8u, symbol Device:L
- removed R3.1: 150k, symbol Device:R
- removed R3.2: 50k, symbol Device:R
- removed R3.3: 200k, symbol Device:R
- removed R3.4: 49.9, symbol Device:R
- removed U3.1: LMR61428, symbol PDU_PROTOTYPE:LMR61428
- added C3.1, C3.3, C3.4: 22u, Capacitor_SMD:C_0805_2012Metric, symbol PowerDistributionUnit-rescue:C-Device
- added C3.2: 1u, Capacitor_SMD:C_0805_2012Metric, symbol PowerDistributionUnit-rescue:C-Device
- added L3.1: 1.5u, Inductor_SMD:L_Taiyo-Yuden_NR-50xx, symbol PowerDistributionUnit-rescue:L-Device
- added R3.1, R3.3: 100k, Resistor_SMD:R_01005_0402Metric, symbol PowerDistributionUnit-rescue:R-Device
- added R3.2: 909k, Resistor_SMD:R_01005_0402Metric, symbol PowerDistributionUnit-rescue:R-Device
- added U3.1: RT4812, Package_TO_SOT_SMD:TSOT-23-8, symbol PDU_PROTOTYPE:RT4812
Connections:
- net labels added: GNDA, Unregulated
- net labels removed: GNDD, UNREGULATED
- wire segments 46 -> 28
