File: MSP430.sch (KiCad schematic (older format))
At the start: 16 parts, among them Q2 CSTCR4M00G15L99, Q2.1 LF_CRYSTAL, U2.1 MSP430F5529IPN

Commit message: updated PDU schematic with footprints
Parts:
- C2.1, C2.10, C2.11, C2.6, C2.8, C2.9: footprint (none) -> Capacitor_SMD:C_0402_1005Metric; symbol Device:C -> PowerDistributionUnit-rescue:C-Device
- C2.2, C2.3: value 22p -> 12p; footprint (none) -> Capacitor_SMD:C_0402_1005Metric; symbol Device:C -> PowerDistributionUnit-rescue:C-Device
- C2.4: footprint (none) -> Capacitor_Tantalum_SMD:CP_EIA-3216-10_Kemet-I; symbol Device:CP1 -> PowerDistributionUnit-rescue:CP1-Device
- C2.5: footprint (none) -> Capacitor_SMD:C_01005_0402Metric; symbol Device:C -> PowerDistributionUnit-rescue:C-Device
- C2.7: footprint (none) -> Capacitor_Tantalum_SMD:CP_EIA-3216-18_Kemet-A; symbol Device:CP1 -> PowerDistributionUnit-rescue:CP1-Device
- Q2.1: footprint (none) -> Crystal:Crystal_SMD_MicroCrystal_MS3V-T1R; symbol Device:Crystal -> PowerDistributionUnit-rescue:Crystal-Device
- R2.1: footprint (none) -> Resistor_SMD:R_01005_0402Metric; symbol Device:R -> PowerDistributionUnit-rescue:R-Device
- U2.1: footprint PN80 -> MSP430F5529:MSP430F5529IPNR
- renumbered Q2 to Q2.2, S1 to S2.1
Connections:
- net labels added: 3.0_SDA_I2C, 3.1_SCL_I2C, SBWCLK, SBWTDIO
- wire segments 122 -> 121
Changed lines of the file:
@@
 $Descr A4 11693 8268
 encoding utf-8
-Sheet 2 5
-Title ""
-Date ""
-Rev ""
-Comp ""
-Comment1 ""
-Comment2 ""
+Sheet 2 6
+Title "Power Distribution Unit - Flat Sat"
+Date "2020-03-08"
+Rev "1"
+Comp "Dalhousie Orbital & Space Systems Lab"
+Comment1 "LORIS"
+Comment2 "Liam JA MacDonald"
 Comment3 ""
 Comment4 ""
@@
 F 0 "U2.1" H 5500 1987 60  0000 C CNN
 F 1 "MSP430F5529IPN" H 5500 1881 60  0000 C CNN
-F 2 "PN80" H 5500 1840 60  0001 C CNN
+F 2 "MSP430F5529:MSP430F5529IPNR" H 5500 1840 60  0001 C CNN
 F 3 "" H 2600 1600 60  0000 C CNN
 	1    2600 1600
@@
 	2700 3300 2600 3300
 $Comp
-L Device:C C2.5
+L PowerDistributionUnit-rescue:C-Device C2.5
 U 1 1 5E2B18E7
 P 1500 3500
 F 0 "C2.5" H 1615 3546 50  0000 L CNN
 F 1 "100n" H 1615 3455 50  0000 L CNN
-F 2 "" H 1538 3350 50  0001 C CNN
+F 2 "Capacitor_SMD:C_01005_0402Metric" H 1538 3350 50  0001 C CNN
 F 3 "~" H 1500 3500 50  0001 C CNN
 	1    1500 3500
@@
 	1500 3650 1500 3700
 $Comp
-L Device:CP1 C2.4
+L PowerDistributionUnit-rescue:CP1-Device C2.4
 U 1 1 5E2B8A75
 P 1000 3500
 F 0 "C2.4" H 1115 3546 50  0000 L CNN
 F 1 "10u" H 1115 3455 50  0000 L CNN
-F 2 "" H 1000 3500 50  0001 C CNN
+F 2 "Capacitor_Tantalum_SMD:CP_EIA-3216-10_Kemet-I" H 1000 3500 50  0001 C CNN
 F 3 "~" H 1000 3500 50  0001 C CNN
 	1    1000 3500
@@
 Connection ~ 1500 3700
 $Comp
-L power:GND #PWR?
+L PowerDistributionUnit-rescue:GND-power #PWR0109
 U 1 1 5E2B94A5
 P 1000 3700
-F 0 "#PWR?" H 1000 3450 50  0001 C CNN
+F 0 "#PWR0109" H 1000 3450 50  0001 C CNN
 F 1 "GND" H 1005 3527 50  0000 C CNN
 F 2 "" H 1000 3700 50  0001 C CNN
@@
 	2600 3400 2000 3400
 $Comp
-L Device:C C2.6
+L PowerDistributionUnit-rescue:C-Device C2.6
 U 1 1 5E2BFB1D
 P 1500 4000
 F 0 "C2.6" H 1615 4046 50  0000 L CNN
 F 1 "470n" H 1615 3955 50  0000 L CNN
-F 2 "" H 1538 3850 50  0001 C CNN
+F 2 "Capacitor_SMD:C_0402_1005Metric" H 1538 3850 50  0001 C CNN
 F 3 "~" H 1500 4000 50  0001 C CNN
 	1    1500 4000
@@
 	1500 3850 1500 3900
 $Comp
-L power:GND #PWR?
+L PowerDistributionUnit-rescue:GND-power #PWR0110
 U 1 1 5E2C3B46
 P 1500 4100
-F 0 "#PWR?" H 1500 3850 50  0001 C CNN
+F 0 "#PWR0110" H 1500 3850 50  0001 C CNN
 F 1 "GND" H 1505 3927 50  0000 C CNN
 F 2 "" H 1500 4100 50  0001 C CNN
@@
 $EndComp
 $Comp
-L Device:Crystal Q2.1
+L PowerDistributionUnit-rescue:Crystal-Device Q2.1
 U 1 1 5E274E19
 P 1500 2850
 F 0 "Q2.1" V 1454 2981 50  0000 L CNN
 F 1 "LF_CRYSTAL" V 1545 2981 50  0000 L CNN
-F 2 "" H 1500 2850 50  0001 C CNN
+F 2 "Crystal:Crystal_SMD_MicroCrystal_MS3V-T1R" H 1500 2850 50  0001 C CNN
 F 3 "~" H 1500 2850 50  0001 C CNN
 	1    1500 2850
@@
 $EndComp
 $Comp
-L Device:C C2.2
+L PowerDistributionUnit-rescue:C-Device C2.2
 U 1 1 5E27C34A
 P 1000 2700
 F 0 "C2.2" V 748 2700 50  0000 C CNN
-F 1 "22p" V 839 2700 50  0000 C CNN
-F 2 "" H 1038 2550 50  0001 C CNN
+F 1 "12p" V 839 2700 50  0000 C CNN
+F 2 "Capacitor_SMD:C_0402_1005Metric" H 1038 2550 50  0001 C CNN
 F 3 "~" H 1000 2700 50  0001 C CNN
 	1    1000 2700
@@
 $EndComp
 $Comp
-L Device:C C2.3
+L PowerDistributionUnit-rescue:C-Device C2.3
 U 1 1 5E27C549
 P 1000 3000
 F 0 "C2.3" V 800 3150 50  0000 C CNN
-F 1 "22p" V 900 3150 50  0000 C CNN
-F 2 "" H 1038 2850 50  0001 C CNN
+F 1 "12p" V 900 3150 50  0000 C CNN
+F 2 "Capacitor_SMD:C_0402_1005Metric" H 1038 2850 50  0001 C CNN
 F 3 "~" H 1000 3000 50  0001 C CNN
 	1    1000 3000
@@
 	2600 2800 2100 2800
 $Comp
-L Device:C C2.1
+L PowerDistributionUnit-rescue:C-Device C2.1
 U 1 1 5E284BFD
 P 650 2850
 F 0 "C2.1" H 650 2750 50  0000 L CNN
 F 1 "100n" H 650 2650 50  0000 L CNN
-F 2 "" H 688 2700 50  0001 C CNN
+F 2 "Capacitor_SMD:C_0402_1005Metric" H 688 2700 50  0001 C CNN
 F 3 "~" H 650 2850 50  0001 C CNN
 	1    650  2850
@@
 	2600 2600 2650 2600
 $Comp
-L Device:C C2.8
+L PowerDistributionUnit-rescue:C-Device C2.8
 U 1 1 5E29DC13
 P 9150 4800
 F 0 "C2.8" H 9265 4846 50  0000 L CNN
 F 1 "100n" H 9265 4755 50  0000 L CNN
-F 2 "" H 9188 4650 50  0001 C CNN
+F 2 "Capacitor_SMD:C_0402_1005Metric" H 9188 4650 50  0001 C CNN
 F 3 "~" H 9150 4800 50  0001 C CNN
 	1    9150 4800
@@
 	650  3150 850  3150
 $Comp
-L power:GND #PWR?
+L PowerDistributionUnit-rescue:GND-power #PWR0111
 U 1 1 5E2A3AD1
 P 650 3150
-F 0 "#PWR?" H 650 2900 50  0001 C CNN
+F 0 "#PWR0111" H 650 2900 50  0001 C CNN
 F 1 "GND" H 655 2977 50  0000 C CNN
 F 2 "" H 650 3150 50  0001 C CNN
@@
 	850  3000 850  3150
 $Comp
-L PowerDistributionUnit-rescue:MURATA-FILTER_CSTCR-MSP-EXP430F5529LP-eagle-import Q2
+L PowerDistributionUnit-rescue:MURATA-FILTER_CSTCR-MSP-EXP430F5529LP-eagle-import Q?
 U 1 1 5E2A7203
 P 9500 2600
-AR Path="/5E2A7203" Ref="Q2"  Part="1"
-AR Path="/5E2222F5/5E2A7203" Ref="Q2"  Part="1"
-F 0 "Q2" H 9500 2886 59  0000 C CNN
+AR Path="/5E2A7203" Ref="Q?"  Part="1"
+AR Path="/5E2222F5/5E2A7203" Ref="Q2.2"  Part="1"
+F 0 "Q2.2" H 9500 2886 59  0000 C CNN
 F 1 "CSTCR4M00G15L99" H 9500 2781 59  0000 C CNN
 F 2 "" H 9500 2600 50  0001 C CNN
@@
 $EndComp
 Wire Wire Line
-	8350 2500 8400 2500
-Wire Wire Line
 	8350 2600 8400 2600
 Connection ~ 9200 2600
@@
 	9800 2600 9950 2600
 $Comp
-L power:GND #PWR?
+L PowerDistributionUnit-rescue:GND-power #PWR0112
 U 1 1 5E2BDD0E
 P 9500 2900
-F 0 "#PWR?" H 9500 2650 50  0001 C CNN
+F 0 "#PWR0112" H 9500 2650 50  0001 C CNN
 F 1 "GND" H 9650 2800 50  0000 C CNN
 F 2 "" H 9500 2900 50  0001 C CNN
@@
 	8400 2600 9200 2600
 $Comp
-L power:GND #PWR?
+L PowerDistributionUnit-rescue:GND-power #PWR0113
 U 1 1 5E2C5347
 P 8900 2800
-F 0 "#PWR?" H 8900 2550 50  0001 C CNN
+F 0 "#PWR0113" H 8900 2550 50  0001 C CNN
 F 1 "GND" H 8905 2627 50  0000 C CNN
 F 2 "" H 8900 2800 50  0001 C CNN
@@
 	8400 2800 8900 2800
 $Comp
-L Device:C C2.10
+L PowerDistributionUnit-rescue:C-Device C2.10
 U 1 1 5E2CC4D8
 P 9950 3350
 F 0 "C2.10" H 10065 3396 50  0000 L CNN
 F 1 "220n" H 10065 3305 50  0000 L CNN
-F 2 "" H 9988 3200 50  0001 C CNN
+F 2 "Capacitor_SMD:C_0402_1005Metric" H 9988 3200 50  0001 C CNN
 F 3 "~" H 9950 3350 50  0001 C CNN
 	1    9950 3350
@@
 	9950 3200 9950 3250
 $Comp
-L Device:C C2.9
+L PowerDistributionUnit-rescue:C-Device C2.9
 U 1 1 5E2D46E3
 P 9500 3350
 F 0 "C2.9" H 9615 3396 50  0000 L CNN
 F 1 "220n" H 9615 3305 50  0000 L CNN
-F 2 "" H 9538 3200 50  0001 C CNN
+F 2 "Capacitor_SMD:C_0402_1005Metric" H 9538 3200 50  0001 C CNN
 F 3 "~" H 9500 3350 50  0001 C CNN
 	1    9500 3350
@@
 Connection ~ 9500 3500
 $Comp
-L Device:CP1 C2.7
+L PowerDistributionUnit-rescue:CP1-Device C2.7
 U 1 1 5E2E0247
 P 8800 3850
 F 0 "C2.7" H 8915 3896 50  0000 L CNN
 F 1 "4u" H 8915 3805 50  0000 L CNN
-F 2 "" H 8800 3850 50  0001 C CNN
+F 2 "Capacitor_Tantalum_SMD:CP_EIA-3216-18_Kemet-A" H 8800 3850 50  0001 C CNN
 F 3 "~" H 8800 3850 50  0001 C CNN
 	1    8800 3850
@@
 	8400 2000 10250 2000
 $Comp
-L PowerDistributionUnit-rescue:PB-MSP-EXP430F5529LP-eagle-import S1
+L PowerDistributionUnit-rescue:PB-MSP-EXP430F5529LP-eagle-import S?
 U 1 1 5E303763
 P 10700 2200
-AR Path="/5E303763" Ref="S1"  Part="1"
+AR Path="/5E303763" Ref="S?"  Part="1"
 AR Path="/5E2222F5/5E303763" Ref="S2.1"  Part="1"
 F 0 "S2.1" H 10743 2253 59  0000 L CNN
@@
 $EndComp
 $Comp
-L Device:C C2.11
+L PowerDistributionUnit-rescue:C-Device C2.11
 U 1 1 5E30880D
 P 10250 2150
 F 0 "C2.11" H 10300 2250 50  0000 L CNN
 F 1 "1n" H 10365 2105 50  0000 L CNN
-F 2 "" H 10288 2000 50  0001 C CNN
+F 2 "Capacitor_SMD:C_0402_1005Metric" H 10288 2000 50  0001 C CNN
 F 3 "~" H 10250 2150 50  0001 C CNN
 	1    10250 2150
@@
 	10700 2400 10700 2350
 Connection ~ 10700 2400
-$Comp
-L power:GND #PWR?
-U 1 1 5E31A3E5
-P 10700 2400
-F 0 "#PWR?" H 10700 2150 50  0001 C CNN
-F 1 "GND" H 10705 2227 50  0000 C CNN
-F 2 "" H 10700 2400 50  0001 C CNN
-F 3 "" H 10700 2400 50  0001 C CNN
-	1    10700 2400
-	1    0    0    -1
-$EndComp
 Wire Wire Line
 	10700 2000 10700 1850
@@
 Wire Notes Line
 	10150 1200 10150 2650
-Wire Notes Line
-	10150 2650 10950 2650
 Wire Notes Line
 	10950 2650 10950 1200
@@
 5V
 $Comp
-L Device:R R2.1
+L PowerDistributionUnit-rescue:R-Device R2.1
 U 1 1 5E31AD4F
 P 10700 1700
 F 0 "R2.1" H 10770 1746 50  0000 L CNN
-F 1 "47k" H 10770 1655 50  0000 L CNN
-F 2 "" V 10630 1700 50  0001 C CNN
+F 1 "47k" V 10700 1650 50  0000 L CNN
+F 2 "Resistor_SMD:R_01005_0402Metric" V 10630 1700 50  0001 C CNN
 F 3 "~" H 10700 1700 50  0001 C CNN
 	1    10700 1700
@@
 3.3V_MSP
 $Comp
-L power:GNDD #PWR?
+L PowerDistributionUnit-rescue:GNDD-power #PWR0115
 U 1 1 5E43CA61
 P 8800 4100
-F 0 "#PWR?" H 8800 3850 50  0001 C CNN
+F 0 "#PWR0115" H 8800 3850 50  0001 C CNN
 F 1 "GNDD" H 8804 3945 50  0000 C CNN
 F 2 "" H 8800 4100 50  0001 C CNN
@@
 Connection ~ 8800 4100
 $Comp
-L power:GNDD #PWR?
+L PowerDistributionUnit-rescue:GNDD-power #PWR0116
 U 1 1 5E443F01
 P 9500 3600
-F 0 "#PWR?" H 9500 3350 50  0001 C CNN
+F 0 "#PWR0116" H 9500 3350 50  0001 C CNN
 F 1 "GNDD" H 9504 3445 50  0000 C CNN
 F 2 "" H 9500 3600 50  0001 C CNN
@@
 $EndComp
 $Comp
-L power:GNDD #PWR?
+L PowerDistributionUnit-rescue:GNDD-power #PWR0117
 U 1 1 5E444A85
 P 9950 3600
-F 0 "#PWR?" H 9950 3350 50  0001 C CNN
+F 0 "#PWR0117" H 9950 3350 50  0001 C CNN
 F 1 "GNDD" H 9954 3445 50  0000 C CNN
 F 2 "" H 9950 3600 50  0001 C CNN
@@
 Wire Wire Line
 	9950 3600 9950 3650
+Wire Notes Line
+	10150 2650 10950 2650
+$Comp
+L PowerDistributionUnit-rescue:GNDD-power #PWR?
+U 1 1 5E880752
+P 10700 2400
+F 0 "#PWR?" H 10700 2150 50  0001 C CNN
+F 1 "GNDD" H 10704 2245 50  0000 C CNN
+F 2 "" H 10700 2400 50  0001 C CNN
+F 3 "" H 10700 2400 50  0001 C CNN
+	1    10700 2400
+	1    0    0    -1
+$EndComp
+Text HLabel 8400 2500 2    50   Input ~ 0
+SBWCLK
+Text HLabel 9400 2000 1    50   Input ~ 0
+SBWTDIO
+Text HLabel 2600 5200 0    50   Input ~ 0
+3.0_SDA_I2C
+Text HLabel 2600 5300 0    50   Output ~ 0
+3.1_SCL_I2C
 $EndSCHEMATC
