File: SubsystemLoadSwitches.sch (KiCad schematic (older format))
At the start: 28 parts

Commit message: updated PDU schematic with footprints
Parts:
- C5.1, C5.2, C5.3, C5.4, C5.5, C5.6, C5.7, C5.8: renamed from C?; footprint (none) -> Capacitor_SMD:C_0805_2012Metric
- R5.1, R5.4: renamed from R?; value TBD -> 3.57m
- R5.10, R5.12, R5.5, R5.7, R5.8, R5.9: renamed from R?; value R -> 100k; footprint (none) -> Resistor_SMD:R_0402_1005Metric; symbol Device:R -> PowerDistributionUnit-rescue:R-Device
- R5.11, R5.6: renamed from R?; value R -> 100k; footprint (none) -> Resistor_SMD:R_01005_0402Metric; symbol Device:R -> PowerDistributionUnit-rescue:R-Device
- R5.13, R5.14, R5.15, R5.16: renamed from R?; value R -> 20k; footprint (none) -> Resistor_SMD:R_0402_1005Metric
- R5.2: renamed from R?; value TBD -> 14.7m
- R5.3: renamed from R?; value TBD -> 22.9m
- U5.1, U5.2, U5.3, U5.4: renamed from U?; footprint (none) -> TPS2557:TPS2557DRBR
Connections:
- net labels added: PL+, PL-
- net labels removed: PAYLOAD+, PAYLOAD-
- wire segments 58 -> 60
Other:
- moved on the sheet: C5.1, C5.2, C5.3, C5.4
