File: PowerDistributionUnit.sch (KiCad schematic (older format))
At the start: 16 parts, among them J1.1 POWER_PINS, J1.2 UART_PINS

Commit message: updated PDU schematic with footprints
Parts:
- removed R?: R, symbol Device:R
- added J1.3: SBW_PINS, Connector_PinHeader_1.27mm:PinHeader_1x02_P1.27mm_Vertical, symbol PowerDistributionUnit-rescue:Conn_01x02_Male-Connector
- added J1.4: I2C_PINS, Connector_PinHeader_1.27mm:PinHeader_1x02_P1.27mm_Vertical, symbol PowerDistributionUnit-rescue:Conn_01x02_Male-Connector
- added R1.5: 86.6k, Resistor_SMD:R_01005_0402Metric, symbol PowerDistributionUnit-rescue:R-Device
- added R1.8, R1.9: 4.7k, symbol PowerDistributionUnit-rescue:R-Device
- J1.1, J1.2: footprint (none) -> Connector_PinHeader_1.27mm:PinHeader_1x02_P1.27mm_Vertical; symbol Connector:Conn_01x02_Male -> PowerDistributionUnit-rescue:Conn_01x02_Male-Connector
- M1.1, M1.2, M1.4: renamed from M?; value MPMOS-pspice -> PMOS; footprint (none) -> Package_TO_SOT_SMD:SOT-23
- M1.3: renamed from M?; value MNMOS -> NMOS; footprint (none) -> digikey-footprints:SOT-23-3; symbol pspice:MNMOS -> PowerDistributionUnit-rescue:MNMOS-pspice
- R1.1, R1.2, R1.6, R1.7: renamed from R?; value R -> 100k; footprint (none) -> Resistor_SMD:R_01005_0402Metric; symbol Device:R -> PowerDistributionUnit-rescue:R-Device
- R1.3: renamed from R?; value R -> 1M; footprint (none) -> Resistor_SMD:R_01005_0402Metric; symbol Device:R -> PowerDistributionUnit-rescue:R-Device
- R1.4: renamed from R?; value R -> 887k; footprint (none) -> Resistor_SMD:R_01005_0402Metric; symbol Device:R -> PowerDistributionUnit-rescue:R-Device
- SW1.1: renamed from SW?; value SW_Push-Switch -> Inhibit; footprint (none) -> Connector_PinHeader_1.27mm:PinHeader_1x02_P1.27mm_Vertical
- SW1.2: renamed from SW?; value SW_Push-Switch -> Inhibit; footprint (none) -> Connector_PinHeader_1.27mm:PinHeader_1x02_P1.27mm_Vertical_SMD_Pin1Right
- U1.1: renamed from U?; value LTC6995-1-CustomSymbols -> LTC6995; footprint (none) -> Package_TO_SOT_SMD:TSOT-23
Connections:
- net labels added: ACS+, ACS-, I_EPS, OBC+, OBC-, PL+, PL-, RF+, RF-
- wire segments 80 -> 106

Commit message: Near complete Pcbnew file for the PDU PCB. All signal routes are complete, need to add ground and power via's to some ICs and a general review. Also need to add print screen to label the different sections of the PCB.
Parts:
- added J1.10: RF_PINS, PDU_Prototype:SAMTEC-TSM-102-01-X-SH, symbol PowerDistributionUnit-rescue:Conn_01x02_Male-Connector
- added J1.11: EPS_PINS, PDU_Prototype:SAMTEC-TSM-102-01-X-SH, symbol PowerDistributionUnit-rescue:Conn_01x02_Male-Connector
- added J1.12: I_BAT_PINS, PDU_Prototype:SAMTEC-TSM-102-01-X-SH, symbol PowerDistributionUnit-rescue:Conn_01x02_Male-Connector
- added J1.13: I_PV_PINS, PDU_Prototype:SAMTEC-TSM-102-01-X-SH, symbol PowerDistributionUnit-rescue:Conn_01x02_Male-Connector
- added J1.5: 30_Minute_Bypass_Jumpers, PDU_Prototype:SAMTEC-TSM-102-01-X-SH, symbol PowerDistributionUnit-rescue:Conn_01x02_Male-Connector
- added J1.6: Direct_Power_Pins, PDU_Prototype:SAMTEC-TSM-102-01-X-SH, symbol PowerDistributionUnit-rescue:Conn_01x02_Male-Connector
- added J1.7: OBC_PINS, PDU_Prototype:SAMTEC-TSM-102-01-X-SH, symbol PowerDistributionUnit-rescue:Conn_01x02_Male-Connector
- added J1.8: PL_PINS, PDU_Prototype:SAMTEC-TSM-102-01-X-SH, symbol PowerDistributionUnit-rescue:Conn_01x02_Male-Connector
- added J1.9: ACS_PINS, PDU_Prototype:SAMTEC-TSM-102-01-X-SH, symbol PowerDistributionUnit-rescue:Conn_01x02_Male-Connector
- added NT1: Net-Tie_2, NetTie:NetTie-2_SMD_Pad2.0mm, symbol Device:Net-Tie_2
- added TP1.1: SW1_TP, TestPoint:TestPoint_Pad_2.0x2.0mm, symbol Connector:TestPoint
- added TP1.2: SW2_TP, TestPoint:TestPoint_Pad_2.0x2.0mm, symbol Connector:TestPoint
- added TP1.3: LTC_TP, TestPoint:TestPoint_Pad_2.0x2.0mm, symbol Connector:TestPoint
- added TP1.4: OBC_TP, TestPoint:TestPoint_Pad_2.0x2.0mm, symbol Connector:TestPoint
- added TP1.5: PL_TP, TestPoint:TestPoint_Pad_2.0x2.0mm, symbol Connector:TestPoint
- added TP1.6: ACS_TP, TestPoint:TestPoint_Pad_2.0x2.0mm, symbol Connector:TestPoint
- added TP1.7: RF_TP, TestPoint:TestPoint_Pad_2.0x2.0mm, symbol Connector:TestPoint
- J1.1, J1.2, J1.3, J1.4: footprint Connector_PinHeader_1.27mm:PinHeader_1x02_P1.27mm_Vertical -> PDU_Prototype:SAMTEC-TSM-102-01-X-SH
- M1.1, M1.2: footprint Package_TO_SOT_SMD:SOT-23 -> Package_DFN_QFN:DFN-6-1EP_2x2mm_P0.5mm_EP0.61x1.42mm; symbol Main-rescue:MPMOS-pspice -> PowerDistributionUnit-rescue:MPMOS-pspice-Main-rescue
- M1.3: footprint digikey-footprints:SOT-23-3 -> Package_SO:SOIC-8_3.9x4.9mm_P1.27mm
- M1.4: footprint Package_TO_SOT_SMD:SOT-23 -> Package_DFN_QFN:DFN-6-1EP_2x2mm_P0.5mm_EP0.61x1.42mm; symbol LORIS_POWER:MPMOS-pspice -> PowerDistributionUnit-rescue:MPMOS-pspice-LORIS_POWER
- R1.1, R1.2, R1.3, R1.4, R1.5, R1.6, R1.7: footprint Resistor_SMD:R_01005_0402Metric -> Resistor_SMD:R_0402_1005Metric
- R1.8, R1.9: footprint (none) -> Resistor_SMD:R_0402_1005Metric
- SW1.1: footprint Connector_PinHeader_1.27mm:PinHeader_1x02_P1.27mm_Vertical -> Button_Switch_SMD:SW_DIP_SPSTx02_Slide_Copal_CHS-02A_W5.08mm_P1.27mm_JPin; symbol Main-rescue:SW_Push-Switch -> PowerDistributionUnit-rescue:SW_Push-Switch-Main-rescue
- SW1.2: footprint Connector_PinHeader_1.27mm:PinHeader_1x02_P1.27mm_Vertical_SMD_Pin1Right -> Button_Switch_SMD:SW_DIP_SPSTx02_Slide_Copal_CHS-02A_W5.08mm_P1.27mm_JPin; symbol Main-rescue:SW_Push-Switch -> PowerDistributionUnit-rescue:SW_Push-Switch-Main-rescue
- U1.1: footprint Package_TO_SOT_SMD:TSOT-23 -> Package_DFN_QFN:DFN-6-1EP_3x2mm_P0.5mm_EP1.65x1.35mm; symbol Main-rescue:LTC6995-1-CustomSymbols -> PowerDistributionUnit-rescue:LTC6995-1-CustomSymbols-Main-rescue
Connections:
- net labels added: 30_Minute_Output, GNDA-power
- net labels removed: 30_Second_Output
- wire segments 106 -> 133
